File: hardware/EspSocket/EspSocket.sch (KiCad schematic (older format))
At the start: 4 parts, among them J1 Conn_01x08, J2 Conn_01x06, J3 Conn_01x08, P1 esp-socket-12

Commit message: Assign Footprints
Parts:
- J1, J3: footprint (none) -> Connector_PinSocket_2.54mm:PinSocket_1x08_P2.54mm_Vertical
- J2: footprint (none) -> Connector_PinSocket_2.54mm:PinSocket_1x06_P2.54mm_Vertical
- P1: footprint (none) -> esp-socket:esp-socket-12
Changed lines of the file:
@@
 F 0 "P1" H 3525 3315 50  0000 C CNN
 F 1 "esp-socket-12" H 3525 3224 50  0000 C CNN
-F 2 "" H 2950 2650 50  0001 C CNN
+F 2 "esp-socket:esp-socket-12" H 2950 2650 50  0001 C CNN
 F 3 "" H 2950 2650 50  0001 C CNN
 	1    3550 2450
@@
 F 0 "J3" H 5350 2950 50  0000 C CNN
 F 1 "Conn_01x08" H 5350 2850 50  0000 C CNN
-F 2 "" H 5400 2400 50  0001 C CNN
+F 2 "Connector_PinSocket_2.54mm:PinSocket_1x08_P2.54mm_Vertical" H 5400 2400 50  0001 C CNN
 F 3 "~" H 5400 2400 50  0001 C CNN
 	1    5400 2400
@@
 F 0 "J1" H 1650 2900 50  0000 L CNN
 F 1 "Conn_01x08" H 1450 2800 50  0000 L CNN
-F 2 "" H 1650 2350 50  0001 C CNN
+F 2 "Connector_PinSocket_2.54mm:PinSocket_1x08_P2.54mm_Vertical" H 1650 2350 50  0001 C CNN
 F 3 "~" H 1650 2350 50  0001 C CNN
 	1    1650 2350
@@
 F 0 "J2" V 3650 4000 50  0000 R CNN
 F 1 "Conn_01x06" V 3550 4150 50  0000 R CNN
-F 2 "" H 3450 4000 50  0001 C CNN
+F 2 "Connector_PinSocket_2.54mm:PinSocket_1x06_P2.54mm_Vertical" H 3450 4000 50  0001 C CNN
 F 3 "~" H 3450 4000 50  0001 C CNN
 	1    3450 4000
