File: hardware/EspSocket/EspSocket.kicad_pcb (KiCad board)
At the start: 2 copper layers, 4 parts, among them J1 Conn_01x08, J2 Conn_01x06, J3 Conn_01x08, P1 esp-socket-12

Commit message: Try adding some artwork
Parts:
- added G***: LOGO, esp-socket:drpep_F_Silk, F.Cu at (147.6, 107.4)
- added GRef: LOGO, esp-socket:drpep_F_Mask, B.Cu at (147.6, 106.5)

Commit message: move art up
Parts:
- moved GRef 4.91 mm to (147.6, 101.6)
- moved G*** 4.81 mm to (148.1, 102.6)
Changed lines of the file:
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@@
   )
   (module esp-socket:drpep_F_Silk (layer F.Cu)
-    (at 147.61464 107.42168)
+    (at 148.0693 102.63632)
     (fp_text reference G*** (at 0 0) (layer F.SilkS) hide
       (effects (font (size 1.524 1.524) (thickness 0.3)))
@@
   )
   (module esp-socket:drpep_F_Mask (layer B.Cu)
-    (at 147.64766 106.50728)
+    (at 147.61464 101.59746)
     (fp_text reference GRef (at 0 0) (layer F.SilkS) hide
       (effects (font (size 1.524 1.524) (thickness 0.3)))
